File: hardware/uv-light-v3.kicad_sch (KiCad schematic)
At the start: 20 parts, among them P1 CON-SENSOR2, P2 DEBUG, P3 BOOT, U1 XMC1100, U2 AS7331, U3 DRILL, U4 DRILL, U5 DRILL, U6 DRILL

Commit message: first pcb layout
Connections:
- net READY: now also U1.14 (P1.0_IHO); no longer U1.21 (P0.12_IO)
- net SCL: now also RP2.8 (R1); no longer RP2.5 (R4)
- net SDA: now also RP2.5 (R4); no longer RP2.8 (R1)
- net SYN: now also U1.13 (P1.1_IHO); no longer U1.20 (P0.9_IO)
- no-connect marks 12 -> 13
Other:
- moved on the sheet: RP2
Changed lines of the file:
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@@
   )
   (no_connect (at 118.11 137.16))
+  (no_connect (at 118.11 77.47))
   (no_connect (at 189.23 83.82))
+  (no_connect (at 118.11 72.39))
   (no_connect (at 191.77 83.82))
+  (no_connect (at 118.11 80.01))
   (no_connect (at 118.11 134.62))
   (no_connect (at 118.11 149.86))
-  (no_connect (at 118.11 107.95))
   (no_connect (at 118.11 142.24))
   (no_connect (at 118.11 113.03))
   (no_connect (at 118.11 115.57))
   (no_connect (at 118.11 144.78))
-  (no_connect (at 118.11 110.49))
   (no_connect (at 118.11 67.31))
   (wire (pts (xy 250.19 80.645) (xy 241.935 80.645))
@@
     (stroke (width 0) (type default) (color 0 0 0 0))
   )
-  (wire (pts (xy 113.03 80.01) (xy 118.11 80.01))
-    (stroke (width 0) (type default) (color 0 0 0 0))
-  )
   (wire (pts (xy 224.155 113.665) (xy 229.87 113.665))
     (stroke (width 0) (type default) (color 0 0 0 0))
@@
     (stroke (width 0) (type default) (color 0 0 0 0))
   )
+  (wire (pts (xy 114.3 110.49) (xy 118.11 110.49))
+    (stroke (width 0) (type default) (color 0 0 0 0))
+  )
   (wire (pts (xy 46.99 26.67) (xy 46.99 25.4))
     (stroke (width 0) (type default) (color 0 0 0 0))
@@
     (stroke (width 0) (type default) (color 0 0 0 0))
   )
+  (wire (pts (xy 114.3 107.95) (xy 118.11 107.95))
+    (stroke (width 0) (type default) (color 0 0 0 0))
+  )
   (wire (pts (xy 250.19 93.345) (xy 250.19 96.52))
     (stroke (width 0) (type default) (color 0 0 0 0))
@@
   )
   (wire (pts (xy 86.36 147.32) (xy 86.36 146.05))
-    (stroke (width 0) (type default) (color 0 0 0 0))
-  )
-  (wire (pts (xy 113.03 77.47) (xy 118.11 77.47))
     (stroke (width 0) (type default) (color 0 0 0 0))
   )
@@
     )
   )
-  (global_label "SYN" (shape input) (at 113.03 77.47 180) (fields_autoplaced)
+  (global_label "SYN" (shape input) (at 114.3 110.49 180) (fields_autoplaced)
     (effects (font (size 1.2 1.2)) (justify right))
-    (property "Intersheet References" "${INTERSHEET_REFS}" (id 0) (at 107.4054 77.395 0)
+    (property "Intersheet References" "${INTERSHEET_REFS}" (id 0) (at 108.6754 110.415 0)
       (effects (font (size 1.2 1.2)) (justify right) hide)
     )
@@
     )
   )
-  (global_label "READY" (shape input) (at 113.03 80.01 180) (fields_autoplaced)
+  (global_label "READY" (shape input) (at 114.3 107.95 180) (fields_autoplaced)
     (effects (font (size 1.2 1.2)) (justify right))
-    (property "Intersheet References" "${INTERSHEET_REFS}" (id 0) (at 105.2911 79.935 0)
+    (property "Intersheet References" "${INTERSHEET_REFS}" (id 0) (at 106.5611 107.875 0)
       (effects (font (size 1.2 1.2)) (justify right) hide)
     )
@@
     (pin "1")
   )
-  (symbol (lib_name "R_PACK4_1") (lib_id "tinkerforge:R_PACK4") (at 185.42 78.74 270) (unit 1)
-    (in_bom yes) (on_board yes)
-    (property "Reference" "RP2" (id 0) (at 196.85 78.74 0)
+  (symbol (lib_name "R_PACK4_1") (lib_id "tinkerforge:R_PACK4") (at 195.58 78.74 90) (mirror x) (unit 1)
+    (in_bom yes) (on_board yes)
+    (property "Reference" "RP2" (id 0) (at 184.15 78.74 0)
       (effects (font (size 1.016 1.016)))
     )
-    (property "Value" "2k2" (id 1) (at 184.15 78.74 0)
+    (property "Value" "2k2" (id 1) (at 196.85 78.74 0)
       (effects (font (size 1.016 1.016)))
     )
-    (property "Footprint" "kicad-libraries:0603X4" (id 2) (at 185.42 78.74 0)
-      (effects (font (size 1.524 1.524)) hide)
-    )
-    (property "Datasheet" "" (id 3) (at 185.42 78.74 0)
-      (effects (font (size 1.524 1.524)))
-    )
+    (property "Footprint" "kicad-libraries:0603X4" (id 2) (at 195.58 78.74 0)
+      (effects (font (size 1.524 1.524)) hide)
+    )
+    (property "Datasheet" "" (id 3) (at 195.58 78.74 0)
+      (effects (font (size 1.524 1.524)))
+    )

Commit message: ready for prototype
Parts:
- RP2: value 2k2 -> 1k
Changed lines of the file:
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@@
       (effects (font (size 1.016 1.016)))
     )
-    (property "Value" "2k2" (id 1) (at 196.85 78.74 0)
+    (property "Value" "1k" (id 1) (at 196.85 78.74 0)
       (effects (font (size 1.016 1.016)))
     )
@@
     )
     (path "/00000000-0000-0000-0000-000055ba021c"
-      (reference "RP2") (unit 1) (value "2k2") (footprint "kicad-libraries:0603X4")
+      (reference "RP2") (unit 1) (value "1k") (footprint "kicad-libraries:0603X4")
     )
     (path "/00000000-0000-0000-0000-00005a86ad72"
